File: hardware/seeknobs5qtpy_22Feb2022.brd (EAGLE design)
At the start: 175.3 x 25.4 mm, 38 parts, among them J1 SJ-3523-SMT, SW1 SPST-6.0MM, SW2 SPST-6.0MM, SW3 SPST-6.0MM, SW4 SPST-6.0MM, U1 ADAFRUIT_QTPYM0

Commit message: more pcb
Parts:
- added SJ1, SJ2: (no value), jumper:SJ
- moved D1 1.30 mm to (3.30, 7.11), turned to 180 degrees
Connections:
- net +3V3: now also SJ1.1, SJ2.1
- net N$9: now also SJ1.2
- net VLED: now also SJ2.2
Routing:
- net +3V3: track 2.11 -> 21.9 mm
- net N$9: track 16.3 -> 33.6 mm
- net VLED: track 180.4 -> 184.4 mm
- net KNOB8: track 40.4 -> 38.9 mm
- net NEOPIXEL: track 151.2 -> 150.0 mm
