File: hardware/seeknobs5qtpy_22Feb2022.sch (EAGLE design)
At the start: 38 parts, among them J1 SJ-3523-SMT, SW1 SPST-6.0MM, SW2 SPST-6.0MM, SW3 SPST-6.0MM, SW4 SPST-6.0MM, U1 ADAFRUIT_QTPYM0

Commit message: more pcb
Parts:
- added SJ1, SJ2: (no value), jumper:SJ
Connections:
- net +3V3: now also SJ1.1, SJ2.1
- net N$9: now also SJ1.2
- net VLED: now also SJ2.2
Changed lines of the file:
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@@
 <part name="GND29" library="supply1" library_urn="urn:adsk.eagle:library:371" deviceset="GND" device=""/>
 <part name="+3V9" library="supply1" library_urn="urn:adsk.eagle:library:371" deviceset="+3V3" device=""/>
-<part name="P+15" library="supply1" library_urn="urn:adsk.eagle:library:371" deviceset="+5V" device=""/>
 <part name="GND44" library="supply1" library_urn="urn:adsk.eagle:library:371" deviceset="GND" device=""/>
 <part name="R1" library="rcl" library_urn="urn:adsk.eagle:library:334" deviceset="R-EU_" device="R0805" package3d_urn="urn:adsk.eagle:package:23553/2" value="33"/>
@@
 <part name="SUPPLY13" library="supply2" library_urn="urn:adsk.eagle:library:372" deviceset="V+" device="" value="VLED"/>
 <part name="SUPPLY14" library="supply2" library_urn="urn:adsk.eagle:library:372" deviceset="V+" device="" value="VLED"/>
+<part name="SUPPLY15" library="supply2" library_urn="urn:adsk.eagle:library:372" deviceset="V+" device="" value="VLED"/>
+<part name="SJ1" library="jumper" library_urn="urn:adsk.eagle:library:252" deviceset="SJ" device="" package3d_urn="urn:adsk.eagle:package:15471/1"/>
+<part name="+3V11" library="supply1" library_urn="urn:adsk.eagle:library:371" deviceset="+3V3" device=""/>
+<part name="SJ2" library="jumper" library_urn="urn:adsk.eagle:library:252" deviceset="SJ" device="" package3d_urn="urn:adsk.eagle:package:15471/1"/>
 </parts>
 <sheets>
@@
 <attribute name="VALUE" x="67.31" y="92.71" size="1.778" layer="96" rot="MR180"/>
 </instance>
-<instance part="P+15" gate="1" x="63.5" y="109.22" smashed="yes">
-<attribute name="VALUE" x="60.96" y="104.14" size="1.778" layer="96" rot="R90"/>
-</instance>
 <instance part="GND44" gate="1" x="236.22" y="50.8" smashed="yes">
 <attribute name="VALUE" x="233.68" y="48.26" size="1.778" layer="96"/>
@@
 <attribute name="VALUE" x="207.01" y="196.85" size="1.778" layer="96"/>
 </instance>
+<instance part="SUPPLY15" gate="1" x="63.5" y="109.22" smashed="yes">
+<attribute name="VALUE" x="62.23" y="110.49" size="1.778" layer="96"/>
+</instance>
+<instance part="SJ1" gate="1" x="154.94" y="198.12" smashed="yes">
+<attribute name="NAME" x="153.67" y="200.406" size="1.778" layer="95"/>
+<attribute name="VALUE" x="152.4" y="194.31" size="1.778" layer="96"/>
+</instance>
+<instance part="+3V11" gate="G$1" x="144.78" y="205.74" smashed="yes" rot="MR0">
+<attribute name="VALUE" x="146.05" y="204.47" size="1.778" layer="96" rot="MR90"/>
+</instance>
+<instance part="SJ2" gate="1" x="154.94" y="205.74" smashed="yes">
+<attribute name="NAME" x="153.67" y="208.026" size="1.778" layer="95"/>
+<attribute name="VALUE" x="152.4" y="201.93" size="1.778" layer="96"/>
+</instance>
 </instances>
 <busses>
@@
 </net>
 <net name="VLED" class="0">
-<segment>
-<pinref part="U1" gate="U$1" pin="5V"/>
-<wire x1="60.96" y1="99.06" x2="63.5" y2="99.06" width="0.1524" layer="91"/>
-<pinref part="P+15" gate="1" pin="+5V"/>
-<wire x1="63.5" y1="99.06" x2="63.5" y2="106.68" width="0.1524" layer="91"/>
-</segment>
 <segment>
 <pinref part="C3" gate="G$1" pin="1"/>
@@
 <wire x1="193.04" y1="200.66" x2="193.04" y2="198.12" width="0.1524" layer="91"/>
 <pinref part="D1" gate="G$1" pin="A"/>
-<wire x1="177.8" y1="198.12" x2="193.04" y2="198.12" width="0.1524" layer="91"/>
+<wire x1="177.8" y1="198.12" x2="185.42" y2="198.12" width="0.1524" layer="91"/>
 <junction x="193.04" y="198.12"/>
+<pinref part="SJ2" gate="1" pin="2"/>
+<wire x1="185.42" y1="198.12" x2="193.04" y2="198.12" width="0.1524" layer="91"/>
+<wire x1="160.02" y1="205.74" x2="185.42" y2="205.74" width="0.1524" layer="91"/>
+<wire x1="185.42" y1="205.74" x2="185.42" y2="198.12" width="0.1524" layer="91"/>
+<junction x="185.42" y="198.12"/>
 </segment>
 <segment>
 <pinref part="LED2" gate="G$1" pin="VDD"/>
 <pinref part="SUPPLY14" gate="1" pin="V+"/>
+</segment>
+<segment>
+<pinref part="U1" gate="U$1" pin="5V"/>
+<wire x1="60.96" y1="99.06" x2="63.5" y2="99.06" width="0.1524" layer="91"/>
+<wire x1="63.5" y1="99.06" x2="63.5" y2="106.68" width="0.1524" layer="91"/>
+<pinref part="SUPPLY15" gate="1" pin="V+"/>
 </segment>
 </net>
@@
 <pinref part="R4" gate="G$1" pin="2"/>
 <wire x1="203.2" y1="40.64" x2="208.28" y2="40.64" width="0.1524" layer="91"/>
+</segment>
+<segment>
+<pinref part="SJ1" gate="1" pin="1"/>
+<wire x1="149.86" y1="198.12" x2="144.78" y2="198.12" width="0.1524" layer="91"/>
+<pinref part="+3V11" gate="G$1" pin="+3V3"/>
+<wire x1="144.78" y1="203.2" x2="144.78" y2="198.12" width="0.1524" layer="91"/>
+<pinref part="SJ2" gate="1" pin="1"/>
+<wire x1="149.86" y1="205.74" x2="149.86" y2="198.12" width="0.1524" layer="91"/>
+<junction x="149.86" y="198.12"/>
 </segment>
 </net>
@@
 <wire x1="170.18" y1="193.04" x2="170.18" y2="198.12" width="0.1524" layer="91"/>
 <junction x="170.18" y="198.12"/>
-</segment>
-</net>
+<pinref part="SJ1" gate="1" pin="2"/>
+<wire x1="160.02" y1="198.12" x2="165.1" y2="198.12" width="0.1524" layer="91"/>
+<junction x="165.1" y="198.12"/>
+</segment>
+</net>
